Commit message: feat: multi-package update — TF stability, pick state machine, approach navigator, arm control
- slam: tf_republisher/fastlio_odom_to_tf use MultiThreadedExecutor + nice -10 priority
- slam: nav2 params tuning, delayed_cloud_relay nice prefix
- perception: image birth timestamp TF queries, service path map frame output
- perception: byte_tracker_3d cleanup, rviz node refactor, synced subscriber improvements
- perception: intrinsics configs, perception server, grasp service extensions
- cleaner_manager: pick state machine major expansion, target pool/filter improvements
- cleaner_manager: manager node service-based detection, rviz config update
- approach_navigator: navigator major enhancement, depth sensor improvements
- piper_grasp: piper_api_v2 + piper_grasp_node major refactor
- cam_lidar_calibration: removed dead code (feature_extractor, optimizer, pose_selector, visualizer)
- robot_desc: URDF updates across all piper descriptions
- Makefile: new targets, scripts: ros_renice.sh, env setup

Co-Authored-By: Claude Opus 4.6 <noreply@anthropic.com>

File: src/robot_desc/piper_description/urdf/piper_description.xacro (robot description, xacro)
@@ -127,6 +127,6 @@
       xyz="0 0 1" />
     <limit
-      lower="-2.687"
-      upper="2.687"
+      lower="-2.618"
+      upper="2.618"
       effort="100"
       velocity="3.142" />
@@ -199,5 +199,5 @@
     <limit
       lower="0"
-      upper="3.403"
+      upper="3.14"
       effort="100"
       velocity="3.403" />
@@ -269,5 +269,5 @@
       xyz="0 0 1" />
     <limit
-      lower="-3.054"
+      lower="-2.967"
       upper="0"
       effort="100"
@@ -339,6 +339,6 @@
       xyz="0 0 1" />
     <limit
-      lower="-1.780"
-      upper="1.780"
+      lower="-1.745"
+      upper="1.745"
       effort="100"
       velocity="3.927" />
@@ -409,6 +409,6 @@
       xyz="0 0 1" />
     <limit
-      lower="-1.309"
-      upper="1.309"
+      lower="-1.22"
+      upper="1.22"
       effort="100"
       velocity="3.927" />
@@ -479,6 +479,6 @@
       xyz="0 0 1" />
     <limit
-      lower="-2.094"
-      upper="2.094"
+      lower="-2.0944"
+      upper="2.0944"
       effort="100"
       velocity="3.927" />

File: src/robot_desc/piper_description/urdf/piper_description_gazebo.xacro (robot description, xacro)
@@ -104,5 +104,5 @@
     <limit
       lower="-2.618"
-      upper="2.168"
+      upper="2.618"
       effort="100"
       velocity="5" />

File: src/robot_desc/piper_description/urdf/piper_description_left.xacro (robot description, xacro)
@@ -141,5 +141,5 @@
         <child link="${namespace}/link3" />
         <axis xyz="0 0 1" />
-        <limit lower="-2.697" upper="0" effort="100" velocity="3" />
+        <limit lower="-2.967" upper="0" effort="100" velocity="3" />
     </joint>
     <link name="${namespace}/link4">
@@ -178,5 +178,5 @@
         <child link="${namespace}/link4" />
         <axis xyz="0 0 1" />
-        <limit lower="-1.832" upper="1.832" effort="100" velocity="3" />
+        <limit lower="-1.745" upper="1.745" effort="100" velocity="3" />
     </joint>
     <link name="${namespace}/link5">
@@ -252,5 +252,5 @@
         <child link="${namespace}/link6" />
         <axis xyz="0 0 1" />
-        <limit lower="-3.14" upper="3.14" effort="100" velocity="3" />
+        <limit lower="-2.0944" upper="2.0944" effort="100" velocity="3" />
     </joint>
     <link name="${namespace}/link7">
@@ -289,5 +289,5 @@
         <child link="${namespace}/link7" />
         <axis xyz="0 0 -1" />
-        <limit lower="0" upper="0.05" effort="10" velocity="1" />
+        <limit lower="0" upper="0.035" effort="10" velocity="1" />
     </joint>
     <link name="${namespace}/link8">
@@ -326,5 +326,5 @@
         <child link="${namespace}/link8" />
         <axis xyz="0 0 1" />
-        <limit lower="-0.05" upper="0" effort="10" velocity="1" />
+        <limit lower="-0.035" upper="0" effort="10" velocity="1" />
     </joint>
 </xacro:macro>

File: src/robot_desc/piper_description/urdf/piper_description_right.xacro (robot description, xacro)
@@ -141,5 +141,5 @@
         <child link="${namespace}/link3" />
         <axis xyz="0 0 1" />
-        <limit lower="-2.697" upper="0" effort="100" velocity="3" />
+        <limit lower="-2.967" upper="0" effort="100" velocity="3" />
     </joint>
     <link name="${namespace}/link4">
@@ -178,5 +178,5 @@
         <child link="${namespace}/link4" />
         <axis xyz="0 0 1" />
-        <limit lower="-1.832" upper="1.832" effort="100" velocity="3" />
+        <limit lower="-1.745" upper="1.745" effort="100" velocity="3" />
     </joint>
     <link name="${namespace}/link5">
@@ -253,5 +253,5 @@
         <child link="${namespace}/link6" />
         <axis xyz="0 0 1" />
-        <limit lower="-3.14" upper="3.14" effort="100" velocity="3" />
+        <limit lower="-2.0944" upper="2.0944" effort="100" velocity="3" />
     </joint>
     <link name="${namespace}/link7">
@@ -290,5 +290,5 @@
         <child link="${namespace}/link7" />
         <axis xyz="0 0 -1" />
-        <limit lower="0" upper="0.05" effort="10" velocity="1" />
+        <limit lower="0" upper="0.035" effort="10" velocity="1" />
     </joint>
     <link name="${namespace}/link8">
@@ -327,5 +327,5 @@
         <child link="${namespace}/link8" />
         <axis xyz="0 0 1" />
-        <limit lower="-0.05" upper="0" effort="10" velocity="1" />
+        <limit lower="-0.035" upper="0" effort="10" velocity="1" />
     </joint>
 </xacro:macro>

File: src/robot_desc/piper_description/urdf/piper_description_with_camera.xacro (robot description, xacro)
@@ -140,5 +140,5 @@
         <child link="link3" />
         <axis xyz="0 0 1" />
-        <limit lower="-2.697" upper="0" effort="100" velocity="3" />
+        <limit lower="-2.967" upper="0" effort="100" velocity="3" />
     </joint>
     <link name="link4">
@@ -177,5 +177,5 @@
         <child link="link4" />
         <axis xyz="0 0 1" />
-        <limit lower="-1.832" upper="1.832" effort="100" velocity="3" />
+        <limit lower="-1.745" upper="1.745" effort="100" velocity="3" />
     </joint>
     <link name="link5">
@@ -251,5 +251,5 @@
         <child link="link6" />
         <axis xyz="0 0 1" />
-        <limit lower="-3.14" upper="3.14" effort="100" velocity="3" />
+        <limit lower="-2.0944" upper="2.0944" effort="100" velocity="3" />
     </joint>
     <link name="link7">
@@ -288,5 +288,5 @@
         <child link="link7" />
         <axis xyz="0 0 -1" />
-        <limit lower="0" upper="0.05" effort="10" velocity="1" />
+        <limit lower="0" upper="0.035" effort="10" velocity="1" />
     </joint>
     <link name="link8">
@@ -325,5 +325,5 @@
         <child link="link8" />
         <axis xyz="0 0 1" />
-        <limit lower="-0.05" upper="0" effort="10" velocity="1" />
+        <limit lower="-0.035" upper="0" effort="10" velocity="1" />
     </joint>
 </robot>

File: src/robot_desc/piper_description/urdf/piper_description_with_camera_left.xacro (robot description, xacro)
@@ -141,5 +141,5 @@
         <child link="${namespace}/link3" />
         <axis xyz="0 0 1" />
-        <limit lower="-2.697" upper="0" effort="100" velocity="3" />
+        <limit lower="-2.967" upper="0" effort="100" velocity="3" />
     </joint>
     <link name="${namespace}/link4">
@@ -178,5 +178,5 @@
         <child link="${namespace}/link4" />
         <axis xyz="0 0 1" />
-        <limit lower="-1.832" upper="1.832" effort="100" velocity="3" />
+        <limit lower="-1.745" upper="1.745" effort="100" velocity="3" />
     </joint>
     <link name="${namespace}/link5">
@@ -252,5 +252,5 @@
         <child link="${namespace}/link6" />
         <axis xyz="0 0 1" />
-        <limit lower="-3.14" upper="3.14" effort="100" velocity="3" />
+        <limit lower="-2.0944" upper="2.0944" effort="100" velocity="3" />
     </joint>
     <link name="${namespace}/link7">
@@ -289,5 +289,5 @@
         <child link="${namespace}/link7" />
         <axis xyz="0 0 -1" />
-        <limit lower="0" upper="0.05" effort="10" velocity="1" />
+        <limit lower="0" upper="0.035" effort="10" velocity="1" />
     </joint>
     <link name="${namespace}/link8">
@@ -326,5 +326,5 @@
         <child link="${namespace}/link8" />
         <axis xyz="0 0 1" />
-        <limit lower="-0.05" upper="0" effort="10" velocity="1" />
+        <limit lower="-0.035" upper="0" effort="10" velocity="1" />
     </joint>
 </xacro:macro>

File: src/robot_desc/piper_description/urdf/piper_description_with_camera_right.xacro (robot description, xacro)
@@ -141,5 +141,5 @@
         <child link="${namespace}/link3" />
         <axis xyz="0 0 1" />
-        <limit lower="-2.697" upper="0" effort="100" velocity="3" />
+        <limit lower="-2.967" upper="0" effort="100" velocity="3" />
     </joint>
     <link name="${namespace}/link4">
@@ -178,5 +178,5 @@
         <child link="${namespace}/link4" />
         <axis xyz="0 0 1" />
-        <limit lower="-1.832" upper="1.832" effort="100" velocity="3" />
+        <limit lower="-1.745" upper="1.745" effort="100" velocity="3" />
     </joint>
     <link name="${namespace}/link5">
@@ -252,5 +252,5 @@
         <child link="${namespace}/link6" />
         <axis xyz="0 0 1" />
-        <limit lower="-3.14" upper="3.14" effort="100" velocity="3" />
+        <limit lower="-2.0944" upper="2.0944" effort="100" velocity="3" />
     </joint>
     <link name="${namespace}/link7">
@@ -289,5 +289,5 @@
         <child link="${namespace}/link7" />
         <axis xyz="0 0 -1" />
-        <limit lower="0" upper="0.05" effort="10" velocity="1" />
+        <limit lower="0" upper="0.035" effort="10" velocity="1" />
     </joint>
     <link name="${namespace}/link8">
@@ -326,5 +326,5 @@
         <child link="${namespace}/link8" />
         <axis xyz="0 0 1" />
-        <limit lower="-0.05" upper="0" effort="10" velocity="1" />
+        <limit lower="-0.035" upper="0" effort="10" velocity="1" />
     </joint>
 </xacro:macro>

File: src/robot_desc/piper_description/urdf/piper_no_gripper_description.xacro (robot description, xacro)
@@ -127,6 +127,6 @@
       xyz="0 0 1" />
     <limit
-      lower="-2.687"
-      upper="2.687"
+      lower="-2.618"
+      upper="2.618"
       effort="100"
       velocity="3.142" />
@@ -199,5 +199,5 @@
     <limit
       lower="0"
-      upper="3.403"
+      upper="3.14"
       effort="100"
       velocity="3.403" />
@@ -269,5 +269,5 @@
       xyz="0 0 1" />
     <limit
-      lower="-3.054"
+      lower="-2.967"
       upper="0"
       effort="100"
@@ -339,6 +339,6 @@
       xyz="0 0 1" />
     <limit
-      lower="-1.780"
-      upper="1.780"
+      lower="-1.745"
+      upper="1.745"
       effort="100"
       velocity="3.927" />
@@ -409,6 +409,6 @@
       xyz="0 0 1" />
     <limit
-      lower="-1.309"
-      upper="1.309"
+      lower="-1.22"
+      upper="1.22"
       effort="100"
       velocity="3.927" />
@@ -479,6 +479,6 @@
       xyz="0 0 1" />
     <limit
-      lower="-2.094"
-      upper="2.094"
+      lower="-2.0944"
+      upper="2.0944"
       effort="100"
       velocity="3.927" />

File: src/robot_desc/piper_description/urdf/piper_no_gripper_description_gazebo.xacro (robot description, xacro)
@@ -104,5 +104,5 @@
     <limit
       lower="-2.618"
-      upper="2.168"
+      upper="2.618"
       effort="100"
       velocity="5" />
